File: reviung39/pcb/reviung39.kicad_pcb (KiCad board)
At the start: 2 copper layers, 248.6 x 104.8 mm, 104 parts, among them SW1 SW_PUSH, SW10 SW_PUSH, SW11 SW_PUSH, SW12 SW_PUSH, SW13 SW_PUSH, SW14 SW_PUSH, SW15 SW_PUSH, SW16 SW_PUSH, SW17 SW_PUSH, SW18 SW_PUSH, SW19 SW_PUSH, SW20 SW_PUSH, SW21 SW_PUSH, SW22 SW_PUSH, SW23 SW_PUSH, SW24 SW_PUSH, SW25 SW_PUSH, SW26 SW_PUSH, SW27 SW_PUSH, SW28 SW_PUSH, SW29 SW_PUSH, SW3 SW_PUSH, SW30 SW_PUSH, SW31 SW_PUSH, SW32 SW_PUSH, SW33 SW_PUSH, SW34 SW_PUSH, SW35 SW_PUSH, SW36 SW_PUSH, SW37 SW_PUSH, SW38 SW_2U_PUSH, SW39 SW_PUSH, SW4 SW_PUSH, SW5 SW_PUSH, SW7 SW_PUSH, SW8 SW_PUSH, SW9 SW_PUSH, U1 ProMicro

Commit message: add pcb, svg and image
Parts:
- added G***: LOGO, _reviung-kbd:REVIUNG39-B-logo, B.Cu at (156.5, 41.9)
- added G***: LOGO, _reviung-kbd:REVIUNG39-FS-logo, F.Cu at (229.0, 102.3)
- added L11: SK6812MINI, _reviung-kbd:LED_SK6812MINI_PLCC4_3.5x3.5mm_P1.75mm, F.Cu at (154.3, 93.9)
- D1, D10, D11, D12, D13, D14, D15, D16, D17, D18, D19, D2, D20, D21, D22, D23, D24, D25, D26, D27, D28, D29, D3, D30, D31, D32, D33, D34, D35, D36, D37, D38, D39, D4, D5, D6, D7, D8, D9: footprint _reviung-kbd:D3_TH_SMD -> _reviung-kbd:D3_SMD_1side; moved to B.Cu
- H1, H10, H11, H2, H3, H4, H5, H6, H7, H8, H9: footprint _riuag-kbd:HOLE -> _reviung-kbd:HOLE
- moved SW13 0.30 mm to (41.2, 89.5)
- moved SW35 0.28 mm to (248.0, 89.4)
- moved SW36 0.25 mm to (267.4, 89.5)
- moved H5 0.25 mm to (106.4, 109.4)
- moved SW39 0.24 mm to (188.3, 123.4)
- moved SW34 0.24 mm to (228.7, 89.3)
- moved SW21 0.24 mm to (202.6, 51.6)
- moved SW1 0.24 mm to (47.9, 52.0)
- moved H11 0.24 mm to (258.9, 96.4)
- moved SW9 0.23 mm to (83.3, 70.5)
- moved SW7 0.23 mm to (44.5, 70.8)
- moved SW33 0.22 mm to (209.3, 89.2)
- moved SW10 0.22 mm to (102.7, 70.4)
- moved H2 0.21 mm to (49.7, 96.4)
- moved SW29 0.21 mm to (244.7, 70.7)
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- renumbered SWe to SW2, SWe to SW6
Routing:
- net VCC: track 489.7 -> 575.6 mm, vias 8 -> 11
- net GND: track 535.8 -> 621.0 mm, vias 37 -> 38
- net Net-(L10-Pad1): track 0.00 -> 76.7 mm, vias 0 -> 1
- net row5: track 196.6 -> 171.4 mm, vias 12 -> 10
- net row0: track 144.1 -> 120.0 mm
- net row1: track 168.7 -> 144.9 mm, vias 4 -> 2
- net row4: track 173.3 -> 149.9 mm, vias 10 -> 8
- net row3: track 148.7 -> 125.7 mm, vias 6 -> 4
- net row2: track 190.7 -> 169.9 mm
- net row6: track 189.7 -> 173.1 mm
- net Net-(L10-Pad3): track 40.9 -> 36.6 mm
- net Net-(D30-Pad2): track 8.03 -> 5.06 mm
- net Net-(D19-Pad2): track 8.11 -> 5.34 mm
- net Net-(D21-Pad2): track 8.06 -> 5.48 mm
- net Net-(D34-Pad2): track 8.07 -> 5.50 mm
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Other:
- board size 248.6 x 104.8 mm -> 247.9 x 104.5 mm
- board text added: "Reviung39 rev1.0 Designed by gtips"
- board text removed: "Reviung39 ver 1.0 PCB Designed by gtips"

Commit message: update pcb ver1.1
Parts:
- U1: footprint _reviung-kbd:ProMicro_v3 -> _reviung-kbd:ProMicro
Other:
- board text added: "Reviung39 rev1.1 Designed by gtips"
- board text removed: "Reviung39 rev1.0 Designed by gtips"
