File: reviung39/pcb/reviung39.sch (KiCad schematic (older format))
At the start: 91 parts, among them SW1 SW_PUSH, SW10 SW_PUSH, SW11 SW_PUSH, SW12 SW_PUSH, SW13 SW_PUSH, SW14 SW_PUSH, SW15 SW_PUSH, SW16 SW_PUSH, SW17 SW_PUSH, SW18 SW_PUSH, SW19 SW_PUSH, SW2 SW_PUSH, SW20 SW_PUSH, SW21 SW_PUSH, SW22 SW_PUSH, SW23 SW_PUSH, SW24 SW_PUSH, SW25 SW_PUSH, SW26 SW_PUSH, SW27 SW_PUSH, SW28 SW_PUSH, SW29 SW_PUSH, SW3 SW_PUSH, SW30 SW_PUSH, SW31 SW_PUSH, SW32 SW_PUSH, SW33 SW_PUSH, SW34 SW_PUSH, SW35 SW_PUSH, SW36 SW_PUSH, SW37 SW_PUSH, SW38 SW_2U_PUSH, SW39 SW_PUSH, SW4 SW_PUSH, SW5 SW_PUSH, SW6 SW_PUSH, SW7 SW_PUSH, SW8 SW_PUSH, SW9 SW_PUSH, U1 ProMicro

Commit message: update pcb ver1.1
Parts:
- U1: footprint _reviung-kbd:ProMicro_v3 -> _reviung-kbd:ProMicro
Changed lines of the file:
@@
 Sheet 1 1
 Title "Reviung39"
-Date "2019-07-11"
-Rev "ver.1"
+Date "2019-09-11"
+Rev "1.1"
 Comp ""
 Comment1 ""
@@
 F 0 "U1" H 2100 3387 60  0000 C CNN
 F 1 "ProMicro" H 2100 3281 60  0000 C CNN
-F 2 "_reviung-kbd:ProMicro_v3" H 2200 1300 60  0001 C CNN
+F 2 "_reviung-kbd:ProMicro" H 2200 1300 60  0001 C CNN
 F 3 "" H 2200 1300 60  0000 C CNN
 	1    2100 2350
