File: reviung39s/pcb/reviung39s.kicad_pcb (KiCad board)
At the start: 2 copper layers, 247.9 x 104.5 mm, 97 parts, among them J1 Conn_01x03_Shielded, SW1 SW_PUSH, SW10 SW_PUSH, SW11 SW_PUSH, SW12 SW_PUSH, SW13 SW_PUSH, SW14 SW_PUSH, SW15 SW_PUSH, SW16 SW_PUSH, SW17 SW_PUSH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

Commit message: update pcb ver1.1
Parts:
- U1: footprint _reviung-kbd:ProMicro_v3 -> _reviung-kbd:ProMicro
