File: reviung39s/pcb/reviung39s.sch (KiCad schematic (older format))
At the start: 91 parts, among them SW1 SW_PUSH, SW10 SW_PUSH, SW11 SW_PUSH, SW12 SW_PUSH, SW13 SW_PUSH, SW14 SW_PUSH, SW15 SW_PUSH, SW16 SW_PUSH, SW17 SW_PUSH, SW18 SW_PUSH, SW19 SW_PUSH, SW2 SW_PUSH, SW20 SW_PUSH, SW21 SW_PUSH, SW22 SW_PUSH, SW23 SW_PUSH, SW24 SW_PUSH, SW25 SW_PUSH, SW26 SW_PUSH, SW27 SW_PUSH, SW28 SW_PUSH, SW29 SW_PUSH, SW3 SW_PUSH, SW30 SW_PUSH, SW31 SW_PUSH, SW32 SW_PUSH, SW33 SW_PUSH, SW34 SW_PUSH, SW35 SW_PUSH, SW36 SW_PUSH, SW37 SW_PUSH, SW38 SW_2U_PUSH, SW39 SW_PUSH, SW4 SW_PUSH, SW5 SW_PUSH, SW6 SW_PUSH, SW7 SW_PUSH, SW8 SW_PUSH, SW9 SW_PUSH, U1 ProMicro

Commit message: add pcb, svg and image
Parts:
- removed L1, L10, L11, L2, L3, L4, L5, L6, L7, L8, L9: SK6812MINI, _reviung-kbd:LED_SK6812MINI_PLCC4_3.5x3.5mm_P1.75mm, symbol _reviung-kbd:SK6812MINI
- added J1: Conn_01x03_Shielded, _reviung-kbd:StripLED_1side, symbol Connector_Generic:Conn_01x03
- D1, D10, D11, D12, D13, D14, D15, D16, D17, D18, D19, D2, D20, D21, D22, D23, D24, D25, D26, D27, D28, D29, D3, D30, D31, D32, D33, D34, D35, D36, D37, D38, D39, D4, D5, D6, D7, D8, D9: footprint _reviung-kbd:D3_SMD_1side -> _reviung-kbd:D3_TH
- SW1, SW10, SW11, SW12, SW13, SW14, SW15, SW16, SW17, SW18, SW19, SW2, SW20, SW21, SW22, SW23, SW24, SW25, SW26, SW27, SW28, SW29, SW3, SW30, SW31, SW32, SW33, SW34, SW35, SW36, SW37, SW39, SW4, SW5, SW6, SW7, SW8, SW9: footprint _reviung-kbd:MXOnly-1U-Hotswap -> _reviung-kbd:MXOnly-1U-NoLED
- SW38: footprint _reviung-kbd:MXOnly-2U-Hotswap-ReversedStabilizers -> _reviung-kbd:MXOnly-2.25U-ReversedStabilizers-NoLED
Connections:
- wire segments 159 -> 86
- no-connect marks 6 -> 5

Commit message: update pcb ver1.1
Parts:
- U1: footprint _reviung-kbd:ProMicro_v3 -> _reviung-kbd:ProMicro
Changed lines of the file:
@@
 EESchema Schematic File Version 4
+LIBS:reviung39s-cache
 EELAYER 29 0
 EELAYER END
@@
 Sheet 1 1
 Title "Reviung39s"
-Date "2019-07-19"
-Rev "ver.1"
+Date "2019-09-11"
+Rev "1.1"
 Comp ""
 Comment1 ""
@@
 F 0 "U1" H 2100 3387 60  0000 C CNN
 F 1 "ProMicro" H 2100 3281 60  0000 C CNN
-F 2 "_reviung-kbd:ProMicro_v3" H 2200 1300 60  0001 C CNN
+F 2 "_reviung-kbd:ProMicro" H 2200 1300 60  0001 C CNN
 F 3 "" H 2200 1300 60  0000 C CNN
 	1    2100 2350
