File: reviung34split/reviung34-split-BOTTOM/reviung34-split-BOTTOM.kicad_pcb (KiCad board)
At the start: 2 copper layers, 100 x 100 mm, 8 parts

Commit message: RJ45_NONAME_8P8C_Horizontal
Redone with very common RJ45_NONAME_8P8C_Horizontal socket's footprint and KiCad 6.0.4.
https://aliexpress.ru/item/32774556179.html
https://aliexpress.ru/item/4001295248605.html
https://aliexpress.ru/item/32694863099.html
https://aliexpress.ru/item/32902228456.html
Other:
- net class Default removed
